File: v0.2/Hardware/Front Panel/Uyue 946-1010/Uyue_946_1010.kicad_pcb (KiCad board)
At the start: 2 copper layers, 96 x 45 mm, 0 parts

Commit message: v0.2: Finished PCBs
Routing:
- added copper zone on B.Cu, net (none)
- added copper zone on F.Cu, net (none)
Other:
- outline, holes or cut-outs redrawn
- board text added: "BACK"
- board text added: "LUNA Embedded"
- board text added: "OK"
- board text added: "Reflow Controller"
Changed lines of the file:
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@@
-(kicad_pcb (version 20171130) (host pcbnew 5.1.9)
+(kicad_pcb (version 20171130) (host pcbnew 5.1.10)
   (general
     (thickness 1.6)
-    (drawings 35)
+    (drawings 51)
     (tracks 0)
     (zones 0)
@@
   (page A4)
   (layers
-    (0 F.Cu signal)
-    (31 B.Cu signal)
+    (0 F.Cu signal hide)
+    (31 B.Cu signal hide)
     (32 B.Adhes user)
     (33 F.Adhes user)
@@
     (last_trace_width 0.25)
     (trace_clearance 0.2)
-    (zone_clearance 0.508)
+    (zone_clearance 0.2)
     (zone_45_only no)
     (trace_min 0.2)
@@
       (outputformat 1)
       (mirror false)
-      (drillshape 1)
+      (drillshape 0)
       (scaleselection 1)
-      (outputdirectory ""))
+      (outputdirectory "Gerbers/"))
   )
   (net 0 "")
@@
     (uvia_dia 0.3)
     (uvia_drill 0.1)
+  )
+  (gr_line (start -41.399998 6.601001) (end -41.4 17.5) (layer Edge.Cuts) (width 0.05))
+  (gr_arc (start -43.000002 -0.002) (end -48.000001 -0.001) (angle -89.98852938) (layer Edge.Cuts) (width 0.05))
+  (gr_arc (start -42.999001 -0.001001) (end -43.000001 -5.001) (angle -89.98852938) (layer Edge.Cuts) (width 0.05))
+  (gr_arc (start -42.999998 6.601001) (end -41.399998 6.601001) (angle -90) (layer Edge.Cuts) (width 0.05))
+  (gr_arc (start -43.001001 -6.599998) (end -43.001001 -4.999998) (angle -90) (layer Edge.Cuts) (width 0.05))
+  (gr_line (start 41.401001 6.599998) (end 41.4 17.5) (layer Edge.Cuts) (width 0.05))
+  (gr_arc (start 43.001001 6.599998) (end 43.001001 4.999998) (angle -90) (layer Edge.Cuts) (width 0.05))
+  (gr_arc (start 43 -6.6) (end 41.4 -6.6) (angle -90) (layer Edge.Cuts) (width 0.05))
+  (gr_arc (start 43.000001 0.001) (end 48 0) (angle -89.98852938) (layer Edge.Cuts) (width 0.05))
+  (gr_arc (start 42.999 0.000001) (end 43 5) (angle -89.98852938) (layer Edge.Cuts) (width 0.05))
+  (gr_arc (start -36.4 17.5) (end -41.4 17.5) (angle -90) (layer Edge.Cuts) (width 0.05))
+  (gr_arc (start 36.4 17.5) (end 36.4 22.5) (angle -90) (layer Edge.Cuts) (width 0.05))
+  (gr_arc (start 36.4 -17.5) (end 41.4 -17.5) (angle -90) (layer Edge.Cuts) (width 0.05))
+  (gr_arc (start -36.4 -17.5) (end -36.4 -22.5) (angle -90) (layer Edge.Cuts) (width 0.05))
+  (gr_line (start -41.4 -17.5) (end -41.4 -6.6) (layer Edge.Cuts) (width 0.05))
+  (gr_line (start 41.4 -17.5) (end 41.4 -6.6) (layer Edge.Cuts) (width 0.05))
+  (gr_poly (pts (xy -26.45 -0.5) (xy -23.55 -0.5) (xy -25 1)) (layer F.Mask) (width 0.1))
+  (gr_poly (pts (xy -23.55 -8.3) (xy -26.45 -8.3) (xy -25 -9.8)) (layer F.Mask) (width 0.1))
+  (gr_text BACK (at 25 0.3) (layer F.Mask)
+    (effects (font (size 1.25 1.25) (thickness 0.25) italic))
+  )
+  (gr_text OK (at 25 -8.95) (layer F.Mask)
+    (effects (font (size 1.25 1.25) (thickness 0.25) italic))
+  )
+  (gr_text "LUNA Embedded" (at 0 17) (layer F.Mask)
+    (effects (font (size 1.5 1.5) (thickness 0.35) italic))
+  )
+  (gr_text "Reflow Controller" (at 0 12) (layer F.Mask)
+    (effects (font (size 2 2) (thickness 0.45)))
   )
   (gr_arc (start -10.87 1.18) (end -11.87 1.18) (angle -90) (layer Edge.Cuts) (width 0.05))
@@
   (gr_circle (center 43 0) (end 44.6 0) (layer Edge.Cuts) (width 0.05))
   (gr_circle (center -43 0) (end -41.4 0) (layer Edge.Cuts) (width 0.05))
-  (gr_arc (start 43 17.5) (end 43 22.5) (angle -90) (layer Edge.Cuts) (width 0.05))
-  (gr_arc (start -43 17.5) (end -48 17.5) (angle -90) (layer Edge.Cuts) (width 0.05))
-  (gr_arc (start -43 -17.5) (end -43 -22.5) (angle -90) (layer Edge.Cuts) (width 0.05))
-  (gr_arc (start 43 -17.5) (end 48 -17.5) (angle -90) (layer Edge.Cuts) (width 0.05))
-  (gr_line (start -48 17.5) (end -48 -17.5) (layer Edge.Cuts) (width 0.05))
-  (gr_line (start -43 22.5) (end 43 22.5) (layer Edge.Cuts) (width 0.05))
-  (gr_line (start 48 17.5) (end 48 -17.5) (layer Edge.Cuts) (width 0.05))
-  (gr_line (start -43 -22.5) (end 43 -22.5) (layer Edge.Cuts) (width 0.05))
+  (gr_line (start -36.4 22.5) (end 36.4 22.5) (layer Edge.Cuts) (width 0.05))
+  (gr_line (start -36.4 -22.5) (end 36.4 -22.5) (layer Edge.Cuts) (width 0.05))
   (gr_circle (center -18.25 -8.95) (end -16.3 -8.95) (layer B.Fab) (width 0.05))
   (gr_circle (center -18.25 0.3) (end -16.3 0.3) (layer B.Fab) (width 0.05))
@@
   (gr_circle (center 18.24 -8.95) (end 20.19 -8.95) (layer B.Fab) (width 0.05))
   (gr_circle (center 183.4 90.7) (end 182.1 89.1) (layer Dwgs.User) (width 0.15))
+  (zone (net 0) (net_name "") (layer F.Cu) (hatch edge 0.508)
+    (connect_pads yes (clearance 0.2))
+    (min_thickness 0.2)
+    (fill yes (arc_segments 32) (thermal_gap 0.2) (thermal_bridge_width 0.3))
+    (polygon
+      (pts
+        (xy 48 -22.5) (xy 48 22.5) (xy -48 22.5) (xy -48 -22.5)
+      )
+    )
+  )
+  (zone (net 0) (net_name "") (layer B.Cu) (hatch edge 0.508)
+    (connect_pads yes (clearance 0.2))
+    (min_thickness 0.2)
+    (fill yes (arc_segments 32) (thermal_gap 0.2) (thermal_bridge_width 0.3))
+    (polygon
+      (pts
+        (xy 48 -22.5) (xy 48 22.5) (xy -48 22.5) (xy -48 -22.5)
+      )
+    )
+  )
 )
