File: v0.2/Hardware/Mainboard/Mainboard.sch (KiCad schematic (older format))
At the start: 53 parts, among them J1 5V, J2 TYPE-C-31-M-12, J3 Debug, J4 TC, J5 S1, J6 S2, Q1 BSS138P, Q2 BSS138P, Q3 BSS138P, SW1 UP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

Commit message: v0.2: Preliminary placement
Connections:
- net labels added: OUT_FAN, OUT_FAN-, OUT_SSR, OUT_SSR-
- net labels removed: OUT1, OUT1-, OUT2, OUT2-
Changed lines of the file:
@@
 	8800 1600 8800 1650
 Text Label 8400 1600 0    50   ~ 0
-OUT1
+OUT_SSR
 Wire Wire Line
 	9250 1300 9250 1350
@@
 	10100 950  9250 950
 Text Label 10100 1350 2    50   ~ 0
-OUT1-
+OUT_SSR-
 $Comp
 L _AKL_Diode:MBR120VLSFT3G D4
@@
 	9250 3450 9250 3650
 Text Label 8400 3250 0    50   ~ 0
-OUT2
+OUT_FAN
 Wire Wire Line
 	9250 2950 9250 3000
@@
 	10100 2600 9250 2600
 Text Label 10100 3000 2    50   ~ 0
-OUT2-
+OUT_FAN-
 $Comp
 L power:GND #PWR01
@@
 Text Label 6800 4800 0    50   ~ 0
 SPI_CS
-Text Label 6800 5600 0    50   ~ 0
-OUT2
-Text Label 6800 5500 0    50   ~ 0
-OUT1
 Text Label 6800 4400 0    50   ~ 0
 BTN_DOWN
@@
 L _AKL_Connector:WJ124-3.81-2P J5
 U 1 1 607B7FA5
-P 10350 1100
-F 0 "J5" H 10350 1200 50  0000 C CNN
-F 1 "S1" H 10350 900 50  0000 C CNN
-F 2 "_AKL_Connector:WJ124-3.81-2P" H 10350 1100 50  0001 C CNN
-F 3 "https://lcsc.com/product-detail/Pluggable-System-Terminal-Block_Ningbo-Kangnex-Elec-WJ124-3-81-2P_C69811.html" H 10350 1100 50  0001 C CNN
-F 4 "WJ124-3.81-2P" H 10350 1100 50  0001 C CNN "MPN"
-	1    10350 1100
-	1    0    0    -1
-$EndComp
-$Comp
-L _AKL_Connector:WJ124-3.81-2P J6
-U 1 1 6098662B
-P 10350 2750
-F 0 "J6" H 10350 2850 50  0000 C CNN
-F 1 "S2" H 10350 2550 50  0000 C CNN
-F 2 "_AKL_Connector:WJ124-3.81-2P" H 10350 2750 50  0001 C CNN
-F 3 "https://lcsc.com/product-detail/Pluggable-System-Terminal-Block_Ningbo-Kangnex-Elec-WJ124-3-81-2P_C69811.html" H 10350 2750 50  0001 C CNN
-F 4 "WJ124-3.81-2P" H 10350 2750 50  0001 C CNN "MPN"
-	1    10350 2750
-	1    0    0    -1
+P 10350 1200
+F 0 "J5" H 10350 1000 50  0000 C CNN
+F 1 "S1" H 10350 1300 50  0000 C CNN
+F 2 "_AKL_Connector:WJ124-3.81-2P" H 10350 1200 50  0001 C CNN
+F 3 "https://lcsc.com/product-detail/Pluggable-System-Terminal-Block_Ningbo-Kangnex-Elec-WJ124-3-81-2P_C69811.html" H 10350 1200 50  0001 C CNN
+F 4 "WJ124-3.81-2P" H 10350 1200 50  0001 C CNN "MPN"
+	1    10350 1200
+	1    0    0    1
 $EndComp
 $Comp
 L _AKL_Connector:WJ124-3.81-2P J1
 U 1 1 6098E68C
-P 1200 1350
-F 0 "J1" H 1200 1450 50  0000 C CNN
-F 1 "5V" H 1200 1150 50  0000 C CNN
-F 2 "_AKL_Connector:WJ124-3.81-2P" H 1200 1350 50  0001 C CNN
-F 3 "https://lcsc.com/product-detail/Pluggable-System-Terminal-Block_Ningbo-Kangnex-Elec-WJ124-3-81-2P_C69811.html" H 1200 1350 50  0001 C CNN
-F 4 "WJ124-3.81-2P" H 1200 1350 50  0001 C CNN "MPN"
-	1    1200 1350
-	-1   0    0    -1
+P 1200 1450
+F 0 "J1" H 1200 1250 50  0000 C CNN
+F 1 "5V" H 1200 1550 50  0000 C CNN
+F 2 "_AKL_Connector:WJ124-3.81-2P" H 1200 1450 50  0001 C CNN
+F 3 "https://lcsc.com/product-detail/Pluggable-System-Terminal-Block_Ningbo-Kangnex-Elec-WJ124-3-81-2P_C69811.html" H 1200 1450 50  0001 C CNN
+F 4 "WJ124-3.81-2P" H 1200 1450 50  0001 C CNN "MPN"
+	1    1200 1450
+	-1   0    0    1
 $EndComp
 $Comp
 L _AKL_Connector:WJ124-3.81-2P J4
 U 1 1 60990BC2
-P 4550 2650
-F 0 "J4" H 4550 2750 50  0000 C CNN
-F 1 "TC" H 4550 2450 50  0000 C CNN
-F 2 "_AKL_Connector:WJ124-3.81-2P" H 4550 2650 50  0001 C CNN
-F 3 "https://lcsc.com/product-detail/Pluggable-System-Terminal-Block_Ningbo-Kangnex-Elec-WJ124-3-81-2P_C69811.html" H 4550 2650 50  0001 C CNN
-F 4 "WJ124-3.81-2P" H 4550 2650 50  0001 C CNN "MPN"
-	1    4550 2650
-	-1   0    0    -1
+P 4550 2750
+F 0 "J4" H 4550 2550 50  0000 C CNN
+F 1 "TC" H 4550 2850 50  0000 C CNN
+F 2 "_AKL_Connector:WJ124-3.81-2P" H 4550 2750 50  0001 C CNN
+F 3 "https://lcsc.com/product-detail/Pluggable-System-Terminal-Block_Ningbo-Kangnex-Elec-WJ124-3-81-2P_C69811.html" H 4550 2750 50  0001 C CNN
+F 4 "WJ124-3.81-2P" H 4550 2750 50  0001 C CNN "MPN"
+	1    4550 2750
+	-1   0    0    1
 $EndComp
 Text Notes 10250 2600 0    50   ~ 0
@@
 Text Label 10550 6900 3    50   ~ 0
 3V3
+$Comp
+L _AKL_Connector:WJ124-3.81-2P J6
+U 1 1 6098662B
+P 10350 2850
+F 0 "J6" H 10350 2650 50  0000 C CNN
+F 1 "S2" H 10350 2950 50  0000 C CNN
+F 2 "_AKL_Connector:WJ124-3.81-2P" H 10350 2850 50  0001 C CNN
+F 3 "https://lcsc.com/product-detail/Pluggable-System-Terminal-Block_Ningbo-Kangnex-Elec-WJ124-3-81-2P_C69811.html" H 10350 2850 50  0001 C CNN
+F 4 "WJ124-3.81-2P" H 10350 2850 50  0001 C CNN "MPN"
+	1    10350 2850
+	1    0    0    1
+$EndComp
+Text Label 6800 5500 0    50   ~ 0
+OUT_SSR
+Text Label 6800 5600 0    50   ~ 0
+OUT_FAN
 $EndSCHEMATC

Commit message: v0.2: Updated placement
Parts:
- SW1, SW2, SW3, SW4: symbol _AKL_Switch:TS-1095-A13B3-D1 -> _AKL_Switch:TS-1095-A135B2-D1; MPN TS-1095-A13B3-D1 -> TS-1095-A135B2-D1
Changed lines of the file:
@@
 $EndComp
 $Comp
-L _AKL_Switch:TS-1095-A13B3-D1 SW1
+L _AKL_Switch:TS-1095-A135B2-D1 SW1
 U 1 1 607B470C
 P 950 5000
-F 0 "SW1" V 1000 5200 50  0000 C CNN
-F 1 "UP" V 900 5200 50  0000 C CNN
+F 0 "SW1" V 900 5200 50  0000 C CNN
+F 1 "UP" V 1000 5200 50  0000 C CNN
 F 2 "Button_Switch_THT:SW_PUSH_6mm_H9.5mm" H 950 5200 50  0001 C CNN
-F 3 "https://lcsc.com/product-detail/Tactile-Switches_Yuandi-TS-1095-A13B3-D1_C493018.html" H 950 5200 50  0001 C CNN
-F 4 "TS-1095-A13B3-D1" H 950 5300 50  0001 C CNN "MPN"
+F 3 "https://lcsc.com/product-detail/Tactile-Switches_Yuandi-TS-1095-A135B2-D1_C782817.html" H 950 5200 50  0001 C CNN
+F 4 "TS-1095-A135B2-D1" H 950 5300 50  0001 C CNN "MPN"
 	1    950  5000
-	0    1    -1   0
+	0    1    1    0
 $EndComp
 $Comp
@@
 F 1 "100" H 9320 4705 50  0000 L CNN
 F 2 "Resistor_SMD:R_0603_1608Metric" H 9250 4750 50  0001 C CNN
-F 3 "https://lcsc.com/product-detail/Chip-Resistor-Surface-Mount_10R-10R-1_C109318.html" H 9250 4750 50  0001 C CNN
+F 3 "https://lcsc.com/product-detail/Chip-Resistor-Surface-Mount_100R-1000-1_C105588.html" H 9250 4750 50  0001 C CNN
 F 4 "RC0603FR-0710RL" H 9250 4750 44  0001 C CNN "MPN"
 	1    9250 4750
@@
 Thermocouple Interface
 $Comp
-L _AKL_Switch:TS-1095-A13B3-D1 SW2
+L _AKL_Switch:TS-1095-A135B2-D1 SW2
 U 1 1 608C10B0
 P 1600 5000
@@
 F 1 "DOWN" V 1550 5200 50  0000 C CNN
 F 2 "Button_Switch_THT:SW_PUSH_6mm_H9.5mm" H 1600 5200 50  0001 C CNN
-F 3 "https://lcsc.com/product-detail/Tactile-Switches_Yuandi-TS-1095-A13B3-D1_C493018.html" H 1600 5200 50  0001 C CNN
-F 4 "TS-1095-A13B3-D1" H 1600 5300 50  0001 C CNN "MPN"
+F 3 "https://lcsc.com/product-detail/Tactile-Switches_Yuandi-TS-1095-A135B2-D1_C782817.html" H 1600 5200 50  0001 C CNN
+F 4 "TS-1095-A135B2-D1" H 1600 5300 50  0001 C CNN "MPN"
 	1    1600 5000
 	0    1    -1   0
 $EndComp
 $Comp
-L _AKL_Switch:TS-1095-A13B3-D1 SW3
+L _AKL_Switch:TS-1095-A135B2-D1 SW3
 U 1 1 608C151B
 P 2250 5000
@@
 F 1 "OK" V 2200 5200 50  0000 C CNN
 F 2 "Button_Switch_THT:SW_PUSH_6mm_H9.5mm" H 2250 5200 50  0001 C CNN
-F 3 "https://lcsc.com/product-detail/Tactile-Switches_Yuandi-TS-1095-A13B3-D1_C493018.html" H 2250 5200 50  0001 C CNN
-F 4 "TS-1095-A13B3-D1" H 2250 5300 50  0001 C CNN "MPN"
+F 3 "https://lcsc.com/product-detail/Tactile-Switches_Yuandi-TS-1095-A135B2-D1_C782817.html" H 2250 5200 50  0001 C CNN
+F 4 "TS-1095-A135B2-D1" H 2250 5300 50  0001 C CNN "MPN"
 	1    2250 5000
 	0    1    -1   0
 $EndComp
 $Comp
-L _AKL_Switch:TS-1095-A13B3-D1 SW4
+L _AKL_Switch:TS-1095-A135B2-D1 SW4
 U 1 1 608C1922
 P 2900 5000
-F 0 "SW4" V 2950 5200 50  0000 C CNN
-F 1 "BACK" V 2850 5200 50  0000 C CNN
+F 0 "SW4" V 2850 5200 50  0000 C CNN
+F 1 "BACK" V 2950 5200 50  0000 C CNN
 F 2 "Button_Switch_THT:SW_PUSH_6mm_H9.5mm" H 2900 5200 50  0001 C CNN
-F 3 "https://lcsc.com/product-detail/Tactile-Switches_Yuandi-TS-1095-A13B3-D1_C493018.html" H 2900 5200 50  0001 C CNN
-F 4 "TS-1095-A13B3-D1" H 2900 5300 50  0001 C CNN "MPN"
+F 3 "https://lcsc.com/product-detail/Tactile-Switches_Yuandi-TS-1095-A135B2-D1_C782817.html" H 2900 5200 50  0001 C CNN
+F 4 "TS-1095-A135B2-D1" H 2900 5300 50  0001 C CNN "MPN"
 	1    2900 5000
-	0    1    -1   0
-$EndComp
-$Comp
+	0    1    1    0
+$EndComp
+$Comp

Commit message: v0.2: Finished PCBs
Connections:
- net BTN_DOWN: now also U3.26 (PA15); no longer U3.7 (PA0)
- net BTN_OK: now also U3.1 (PB9); no longer U3.14 (PA7)
- net BTN_UP: now also U3.27 (PB3); no longer U3.8 (PA1)
- net PWM_BUZZER: now also U3.28 (PB4); no longer U3.18 (PA8)
Changed lines of the file:
@@
 Sheet 1 1
 Title "Reflow Controller"
-Date "2021-04-17"
+Date "2021-05-04"
 Rev "v0.2"
 Comp "LUNAEmbedded.com"
@@
 Text Label 5000 5200 2    50   ~ 0
 I2C_SCL
-Text Label 6800 5200 0    50   ~ 0
-PWM_BUZZER
 Text Label 6800 5000 0    50   ~ 0
 SPI_MISO
@@
 Text Label 6800 4800 0    50   ~ 0
 SPI_CS
-Text Label 6800 4400 0    50   ~ 0
+Text Label 6800 5900 0    50   ~ 0
 BTN_DOWN
-Text Label 6800 4500 0    50   ~ 0
+Text Label 5000 4900 2    50   ~ 0
 BTN_UP
 Text Notes 3100 6750 0    79   Italic 16
@@
 MCU_RXD
 NoConn ~ 6800 4600
-Text Label 6800 5100 0    50   ~ 0
+Text Label 5000 5500 2    50   ~ 0
 BTN_OK
 Text Label 6800 4700 0    50   ~ 0
@@
 Text Notes 6950 4700 0    50   ~ 0
 USART2_RX
-NoConn ~ 6800 5900
-NoConn ~ 5000 5500
+NoConn ~ 6800 4400
+NoConn ~ 6800 5100
 NoConn ~ 5000 5400
 NoConn ~ 5000 5100
-NoConn ~ 5000 5000
-NoConn ~ 5000 4900
+NoConn ~ 6800 5200
+NoConn ~ 6800 4500
 NoConn ~ 5000 4800
 NoConn ~ 5000 4700
@@
 Text Label 6800 5600 0    50   ~ 0
 OUT_FAN
+Text Label 5000 5000 2    50   ~ 0
+PWM_BUZZER
 $EndSCHEMATC
