File: Mainboard/Mainboard.kicad_pcb (KiCad board)
At the start: 2 copper layers, 44 x 44 mm, 50 parts, among them J1 5V, J2 TYPE-C-31-M-12, J3 Debug, J4 TC, J5 S1, J6 S2, Q1 BSS138P, Q2 BSS138P, Q3 BSS138P, SW1 UP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

Commit message: Updated project files to KiCad 10
Other:
- net class 3V3 removed
- net class Default removed
- net class Power removed
- net class USB removed
